Commit message: Merge SCARA simulation and digital twin updates

File: urdf/arm.xacro (robot description, xacro)
@@ -2,7 +2,4 @@
 <robot name="scara" xmlns:xacro="http://www.ros.org/wiki/xacro">
     <!-- Materials -->
-    <material name="scara_wood_brown">
-        <color rgba="0.75 0.52 0.32 1.0"/>
-    </material>
     <material name="scara_mid_blue">
         <color rgba="0.0 0.4 0.8 1.0"/>
@@ -11,32 +8,27 @@
         <color rgba="0.0 0.1 0.4 1.0"/>
     </material>
+    <material name="scara_name_white">
+        <color rgba="0.96 0.96 0.96 1.0"/>
+    </material>
     <material name="scara_light_grey">
         <color rgba="0.7 0.7 0.7 1.0"/>
     </material>
-    <!-- ── WOODEN TABLE BASE PLATFORM ────────────────────────────── -->
-    <link name="table_link">
-        <visual>
-            <origin xyz="0.25 0 -0.10" rpy="0 0 0"/>
-            <geometry>
-                <box size="1.20 0.85 0.20"/>
-            </geometry>
-            <material name="scara_wood_brown"/>
-        </visual>
-        <collision>
-            <origin xyz="0.25 0 -0.10" rpy="0 0 0"/>
-            <geometry>
-                <box size="1.20 0.85 0.20"/>
-            </geometry>
-        </collision>
-        <inertial>
-            <origin xyz="0.25 0 -0.10" rpy="0 0 0"/>
-            <mass value="50.0"/>
-            <inertia ixx="1.0" ixy="0.0" ixz="0.0" iyy="1.0" iyz="0.0" izz="1.0"/>
-        </inertial>
-    </link>
-    <!-- Joint mounting SCARA robot base on top of the wooden table -->
-    <joint name="table_to_base_joint" type="fixed">
-        <origin xyz="0.05 0.08 0.0" rpy="0 0 0"/>
-        <parent link="table_link"/>
+    <!-- ── MOUNT ──────────────────────────────────────────────────────
+         The table, conveyor, bins and cameras now live in worlds/scara_world.sdf.
+         The conveyor runs across the table in front of the robot (like the
+         videos and the SCARA Digital Twin app).
+         The robot is bolted to the table top through a fixed joint to "world"
+         (it used to carry its own table box, which sat half below the ground
+         and was free to tip over).  Values match scripts/scara_scene.py
+         (BASE_XYZ / BASE_YAW): the robot is turned 180 deg so it faces the
+         viewer with the conveyor in front of it. -->
+    <xacro:property name="mount_x" value="0.20"/>
+    <xacro:property name="mount_y" value="0.0"/>
+    <xacro:property name="mount_z" value="0.40"/>
+    <xacro:property name="mount_yaw" value="3.141592653589793"/>
+    <link name="world"/>
+    <joint name="world_to_base_joint" type="fixed">
+        <origin xyz="${mount_x} ${mount_y} ${mount_z}" rpy="0 0 ${mount_yaw}"/>
+        <parent link="world"/>
         <child link="base_link"/>
     </joint>
@@ -108,6 +100,17 @@
             <material name="scara_mid_blue"/>
         </visual>
-        <collision>
-            <origin xyz="-0.059954333 -0.59974857 -0.390000" rpy="0 0 0"/>
+        <!-- raised name plate: same frame and scale as shoulder_link.stl -->
+        <xacro:if value="$(arg name_plate)">
+            <visual name="name_plate">
+                <origin xyz="-0.059954333 -0.059974857 -0.390000" rpy="0 0 0"/>
+                <geometry>
+                    <mesh filename="package://scara_description/meshes/shoulder_name.stl"
+                          scale="0.001 0.001 0.001"/>
+                </geometry>
+                <material name="scara_name_white"/>
+            </visual>
+        </xacro:if>
+        <collision>
+            <origin xyz="-0.059954333 -0.059974857 -0.390000" rpy="0 0 0"/>
             <geometry>
                 <mesh filename="package://scara_description/meshes/shoulder_link.stl"
@@ -194,10 +197,45 @@
         <limit lower="-4.712" upper="4.712" effort="10.0" velocity="1.5"/>
     </joint>
-    <!-- Tool centre point: centre of the gripper finger tips. -->
+    <!-- Tool centre point: centre of the two finger pads (measured from the
+         finger meshes; the old value 0.08 sat on the front edge of the fingers) -->
     <link name="tool0"/>
     <joint name="tool0_joint" type="fixed">
         <parent link="wrist_link"/>
         <child link="tool0"/>
-        <origin xyz="0.08 0 -0.10" rpy="0 0 0"/>
+        <origin xyz="0.0334 0 -0.0985" rpy="0 0 0"/>
+    </joint>
+    <!-- ── ARM CAMERA ───────────────────────────────────────────────
+         camera_link.stl on a bracket at the front of the forearm, beside the
+         wrist, aimed down at the finger pads (70 deg HFOV, 320x240).  It is
+         fixed to the forearm, so turning the wrist never swings it into the
+         forearm or the shoulder link.  Same pose as scripts/scara_scene.py
+         (ARM_CAM_*) and the phone app.  The link frame is the camera frame:
+         +X = viewing direction, +Z = image up. -->
+    <link name="arm_camera_link">
+        <visual>
+            <origin xyz="-0.1405 0 -0.115" rpy="0 0 0"/>
+            <geometry>
+                <mesh filename="package://scara_description/meshes/camera_link.stl"
+                      scale="0.001 0.001 0.001"/>
+            </geometry>
+            <material name="scara_camera_grey">
+                <color rgba="0.13 0.13 0.15 1.0"/>
+            </material>
+        </visual>
+        <visual>
+            <!-- mounting bracket on the wrist housing -->
+            <origin xyz="0.00848 0 -0.01644" rpy="0 -1.71681 0"/>
+            <geometry><box size="0.011 0.032 0.024"/></geometry>
+            <material name="scara_dark_blue"/>
+        </visual>
+        <inertial>
+            <mass value="0.05"/>
+            <inertia ixx="1e-5" ixy="0" ixz="0" iyy="1e-5" iyz="0" izz="1e-5"/>
+        </inertial>
+    </link>
+    <joint name="arm_camera_joint" type="fixed">
+        <parent link="forearm_link"/>
+        <child link="arm_camera_link"/>
+        <origin xyz="0.205 0 0" rpy="0 1.71681 0"/>
     </joint>
     <!-- ── LEFT FINGER ───────────────────────────────── -->
@@ -211,17 +249,18 @@
             <material name="scara_light_grey"/>
         </visual>
-        <collision>
+        <collision name="pad">
+            <origin xyz="0.03185 -0.00485 -0.085" rpy="0 0 0"/>
+            <geometry><box size="0.0919 0.0269 0.02"/></geometry>
+        </collision>
+        <collision name="bar">
+            <origin xyz="-0.00095 -0.00725 -0.0325" rpy="0 0 0"/>
+            <geometry><box size="0.0267 0.0281 0.085"/></geometry>
+        </collision>
+        <inertial>
             <origin xyz="-0.409 -0.0626 -0.2775" rpy="0 0 0"/>
-            <geometry>
-                <mesh filename="package://scara_description/meshes/left_finger_link.stl"
-                      scale="0.001 0.001 0.001"/>
-            </geometry>
-        </collision>
-        <inertial>
-            <origin xyz="-0.409 -0.0626 -0.2775" rpy="0 0 0"/>
-            <mass value="1.0"/>
-            <inertia ixx="0.01" ixy="0.0" ixz="0.0"
-                               iyy="0.01" iyz="0.0"
-                               izz="0.01"/>
+            <mass value="0.2"/>
+            <inertia ixx="0.001" ixy="0.0" ixz="0.0"
+                               iyy="0.001" iyz="0.0"
+                               izz="0.001"/>
         </inertial>
     </link>
@@ -232,5 +271,5 @@
         <child link="left_finger_link"/>
         <axis xyz="0 1 0"/>
-        <limit lower="-0.06" upper="0.0" effort="100.0" velocity="0.5"/>
+        <limit lower="-0.06" upper="0.0" effort="20.0" velocity="0.1"/>
     </joint>
     <!-- ── RIGHT FINGER ──────────────────────────────── -->
@@ -244,17 +283,18 @@
             <material name="scara_light_grey"/>
         </visual>
-        <collision>
+        <collision name="pad">
+            <origin xyz="0.0350 0.00605 -0.085" rpy="0 0 0"/>
+            <geometry><box size="0.0926 0.0251 0.02"/></geometry>
+        </collision>
+        <collision name="bar">
+            <origin xyz="0.00195 0.00825 -0.0325" rpy="0 0 0"/>
+            <geometry><box size="0.0267 0.0267 0.085"/></geometry>
+        </collision>
+        <inertial>
             <origin xyz="-0.409 0.0626 -0.2775" rpy="0 0 0"/>
-            <geometry>
-                <mesh filename="package://scara_description/meshes/right_finger_link.stl"
-                      scale="0.001 0.001 0.001"/>
-            </geometry>
-        </collision>
-        <inertial>
-            <origin xyz="-0.409 0.0626 -0.2775" rpy="0 0 0"/>
-            <mass value="1.0"/>
-            <inertia ixx="0.01" ixy="0.0" ixz="0.0"
-                               iyy="0.01" iyz="0.0"
-                               izz="0.01"/>
+            <mass value="0.2"/>
+            <inertia ixx="0.001" ixy="0.0" ixz="0.0"
+                               iyy="0.001" iyz="0.0"
+                               izz="0.001"/>
         </inertial>
     </link>
@@ -265,5 +305,5 @@
         <child link="right_finger_link"/>
         <axis xyz="0 -1 0"/>
-        <limit lower="-0.06" upper="0.0" effort="100.0" velocity="0.5"/>
+        <limit lower="-0.06" upper="0.0" effort="20.0" velocity="0.1"/>
     </joint>
     <!-- DUMMY JOINT FOR MOVEIT2-->
@@ -309,6 +349,43 @@
 </joint>
     </ros2_control>
-    <gazebo reference="table_link">
-        <material>Gazebo/Wood</material>
+    <!-- High-friction finger pads so pucks are held by friction -->
+    <gazebo reference="left_finger_link">
+        <mu1>1.5</mu1>
+        <mu2>1.5</mu2>
+        <kp>100000.0</kp>
+        <kd>10.0</kd>
+        <minDepth>0.0005</minDepth>
+        <maxVel>0.1</maxVel>
+    </gazebo>
+    <gazebo reference="right_finger_link">
+        <mu1>1.5</mu1>
+        <mu2>1.5</mu2>
+        <kp>100000.0</kp>
+        <kd>10.0</kd>
+        <minDepth>0.0005</minDepth>
+        <maxVel>0.1</maxVel>
+    </gazebo>
+    <!-- Arm camera on the forearm ("SCARA Arm Camera" window) -->
+    <gazebo reference="arm_camera_link">
+        <sensor name="arm_camera" type="camera">
+            <!-- lens on the front face of the camera body -->
+            <pose>0.012 0 0 0 0 0</pose>
+            <always_on>true</always_on>
+            <update_rate>15</update_rate>
+            <visualize>false</visualize>
+            <topic>arm_camera/image</topic>
+            <camera>
+                <horizontal_fov>1.2217</horizontal_fov>
+                <image>
+                    <width>320</width>
+                    <height>240</height>
+                    <format>R8G8B8</format>
+                </image>
+                <clip>
+                    <near>0.02</near>
+                    <far>3.0</far>
+                </clip>
+            </camera>
+        </sensor>
     </gazebo>
     <gazebo>

File: urdf/scara.urdf.xacro (robot description, xacro)
@@ -3,4 +3,8 @@
     <!-- Load Simulated or Real Hardware Interfaces -->
     <xacro:arg name="is_sim" default="true"/>
+    <!-- Raised name on top of the shoulder link (meshes/shoulder_name.stl, made by
+         tools/make_name_mesh.py). The launch files switch it on automatically when
+         that mesh file exists; by hand: xacro scara.urdf.xacro name_plate:=true -->
+    <xacro:arg name="name_plate" default="false"/>
     <xacro:include filename="$(find scara_description)/urdf/arm.xacro" />
 </robot>
